Commit message: sintonizacionPID

File: my_bot/description/robot_core.xacro (robot description, xacro)
@@ -10,9 +10,9 @@
     <xacro:property name="wheel_mass" value="0.03"/>
     <xacro:property name="wheel_offset_x" value="0.02"/>
-    <xacro:property name="wheel_offset_y" value="-0.11"/>
+    <xacro:property name="wheel_offset_y" value="0.11"/>
     <xacro:property name="wheel_offset_z" value="0"/>
     <xacro:property name="caster_wheel_radius" value="0.02"/>
     <xacro:property name="caster_wheel_mass" value="0.03"/>
-    <xacro:property name="caster_wheel_offset_x" value="0.19"/>
+    <xacro:property name="caster_wheel_offset_x" value="0.02"/>
     <!--<xacro:property name="caster_wheel_offset_z" value="${wheel_offset_z - wheel_radius + caster_wheel_radius}"/> -->
     <material name="white">
@@ -65,5 +65,5 @@
         <parent link="base_link"/>
         <child link="left_wheel"/>
-        <origin xyz="0 ${wheel_offset_y} 0" rpy="-${pi/2} 0 0" />
+        <origin xyz="0.195 ${wheel_offset_y} 0" rpy="-${pi/2} 0 0" />
         <axis xyz="0 0 -1"/>
     </joint>
@@ -91,5 +91,5 @@
         <parent link="base_link"/>
         <child link="right_wheel"/>
-        <origin xyz="0 ${-wheel_offset_y} 0" rpy="${pi/2} 0 0" />
+        <origin xyz="0.195 ${-wheel_offset_y} 0" rpy="${pi/2} 0 0" />
         <axis xyz="0 0 1"/>
     </joint>

Commit message: 12/17/22

File: my_bot/description/robot_core.xacro (robot description, xacro)
@@ -66,5 +66,5 @@
         <child link="left_wheel"/>
         <origin xyz="0.195 ${wheel_offset_y} 0" rpy="-${pi/2} 0 0" />
-        <axis xyz="0 0 -1"/>
+        <axis xyz="0 0 1"/>
     </joint>
     <link name="left_wheel">
@@ -92,5 +92,5 @@
         <child link="right_wheel"/>
         <origin xyz="0.195 ${-wheel_offset_y} 0" rpy="${pi/2} 0 0" />
-        <axis xyz="0 0 1"/>
+        <axis xyz="0 0 -1"/>
     </joint>
     <link name="right_wheel">
