Commit message: control remoto

File: my_bot/description/robot.urdf.xacro (robot description, xacro)
@@ -5,4 +5,5 @@
     <xacro:include filename="ros2_control.xacro" />
     <xacro:include filename="robot_core.xacro" />
+    <xacro:include filename="lidar.xacro" />
     <!--<xacro:if value="$(arg use_ros2_control)">
     </xacro:if>

File: my_bot/description/robot_core.xacro (robot description, xacro)
@@ -33,4 +33,12 @@
     <!-- BASE LINK -->
     <link name="base_link">
+    </link>
+    <!-- Base_Footprint Link-->
+    <joint name="base_footprint_joint" type="fixed">
+        <parent link="base_link"/>
+        <child link="base_footprint"/>
+        <origin xyz="0 0 0" rpy="0 0 0"/>
+    </joint>
+    <link name="base_footprint">
     </link>
     <!-- CHASSIS LINK -->
