Commit message: nav2

File: my_bot/description/gazebo_control.xacro (robot description, xacro)
@@ -6,6 +6,6 @@
             <left_joint>left_wheel_joint</left_joint>
             <right_joint>right_wheel_joint</right_joint>
-            <wheel_separation>0.22</wheel_separation>
-            <wheel_diameter>0.0665</wheel_diameter>
+            <wheel_separation>0.255</wheel_separation>
+            <wheel_diameter>0.068</wheel_diameter>
             <!-- Limits -->
             <max_wheel_torque>200</max_wheel_torque>

File: my_bot/description/robot_core.xacro (robot description, xacro)
@@ -5,5 +5,5 @@
     <xacro:property name="chassis_width" value="0.19"/>
     <xacro:property name="chassis_height" value="0.02"/>
-    <xacro:property name="chassis_mass" value="1.335"/>
+    <xacro:property name="chassis_mass" value="2"/>
     <xacro:property name="wheel_radius" value="0.03325"/>
     <xacro:property name="wheel_thickness" value="0.0266"/>
@@ -143,4 +143,18 @@
         </xacro:inertial_sphere>
     </link>
+    <link name="imu_link"/>
+    <joint
+        name="imu_joint"
+        type="fixed">
+        <origin
+        xyz="0.0 0 0.0"
+        rpy="0 -0.07 0" />
+        <parent
+        link="base_link" />
+        <child
+        link="imu_link" />
+        <axis
+        xyz="1 0 0" />
+    </joint>
     <gazebo reference="caster_wheel">
         <material>Gazebo/White</material>

File: my_bot/description/ros2_control.xacro (robot description, xacro)
@@ -6,9 +6,9 @@
                 <param name="left_wheel_name">left_wheel_joint</param>
                 <param name="right_wheel_name">right_wheel_joint</param>
-                <param name="loop_rate">100</param>
+                <param name="loop_rate">30</param>
                 <param name="device">/dev/ttyACM0</param>
                 <param name="baud_rate">115200</param>
-                <param name="timeout">10000</param>
-                <param name="enc_counts_per_rev">620</param>
+                <param name="timeout">5000</param>
+                <param name="enc_counts_per_rev">1300</param>
             </hardware>
             <joint name="left_wheel_joint">
